File: floppy-adapter-2.kicad_sch (KiCad schematic)
At the start: 5 parts, among them J1 Female Floppy Connector, J2 Edge Connector

Commit message: Flip the silkscreen to the other side for the 34-pin connector, finally
Parts:
- J1: footprint Connector_PinHeader_2.54mm:PinHeader_2x17_P2.54mm_Vertical -> EdgeConnectors:Floppy_Connector
